File: hardware/kicad/mcu.kicad_sch (KiCad schematic)
At the start: 19 parts, among them J1 C2, U5 EFM8BB21F16G-C-QSOP24

Commit message: WIP: zone/place fields, lamp chain moved to P2.0-P2.3, power sheet re-flow
Pin sides follow placement (QSOP pins 1-12 power/panel side, 13-24 RF side).
Block diagram and Olimex-style restyle still pending.

Co-Authored-By: Claude Opus 5.5 <noreply@anthropic.com>
Claude-Session: https://claude.ai/code/session_01YRUiF8Vp4242sya9Xyg3TV
Parts:
- C14: Place (none) -> U5.6; Zone (none) -> DIGITAL
- C15: Place (none) -> U5.6 (closest); Zone (none) -> DIGITAL
- J1: Place (none) -> edge; Zone (none) -> DIGITAL
- R13: Place (none) -> U5.7; Zone (none) -> DIGITAL
- R14: Place (none) -> U5.22; Zone (none) -> DIGITAL
- R15: Place (none) -> U5.21; Zone (none) -> DIGITAL
- R16: Place (none) -> U5.20; Zone (none) -> DIGITAL
- R17: Place (none) -> U5.19; Zone (none) -> DIGITAL
- R18: Place (none) -> U5.18; Zone (none) -> DIGITAL
- R19: Place (none) -> U5.17; Zone (none) -> DIGITAL
- R20: Place (none) -> U5.9; Zone (none) -> DIGITAL
- TP1, TP6, TP7, U5: Zone (none) -> DIGITAL
- TP2: value SPARE_P20 -> SPARE_P14; Zone (none) -> DIGITAL
- TP3: value SPARE_P21 -> SPARE_P15; Zone (none) -> DIGITAL
- TP4: value SPARE_P22 -> SPARE_P16; Zone (none) -> DIGITAL
- TP5: value SPARE_P23 -> SPARE_P17; Zone (none) -> DIGITAL
Connections:
- net LED_OE_N: now also U5.9 (P2.3); no longer U5.13 (P1.7)
- net LED_RCK: now also U5.10 (P2.2); no longer U5.14 (P1.6/SCL)
- net LED_SCK: now also U5.11 (P2.1); no longer U5.15 (P1.5/SDA)
- net LED_SER: now also U5.12 (P2.0); no longer U5.16 (P1.4)
- net SPARE_P20 renamed SPARE_P14
- net SPARE_P14: now also U5.16 (P1.4); no longer U5.12 (P2.0)
- net SPARE_P21 renamed SPARE_P15
- net SPARE_P15: now also U5.15 (P1.5/SDA); no longer U5.11 (P2.1)
- net SPARE_P22 renamed SPARE_P16
- net SPARE_P16: now also U5.14 (P1.6/SCL); no longer U5.10 (P2.2)
- net SPARE_P23 renamed SPARE_P17
- net SPARE_P17: now also U5.13 (P1.7); no longer U5.9 (P2.3)
Other:
- note added: "Pins follow placement: QSOP pins 1-12 (analog, debug, lamp chain P2.x) face power/panel,"
- note added: "pins 13-24 (switch control, LNA_EN, FAULT_N) face the RF chain. No control line crosses the MCU."

Commit message: Schematic v0.2: Olimex-style redraw with block diagram
- power/ground only as power symbols (project rails VCOAX, VMAIN, VHOLD, VLED, LNA_VCC)
- wires inside blocks, hierarchical labels + sheet pins between sheets (no global labels)
- Value carries critical parameters, blue design-intent notes, bold italic block titles
- sheet 1: block diagram + wired hierarchy; RF/Panel placeholders with reset-safe pulls
- pull-downs moved to the receiving parts (TPS2553 EN, RF switches), RC filters to the ADC pins
- check.py compares net partitions (catches shorts and splits), generator flags 4-way junctions
- net classes in .kicad_pro (POWER 0.4 mm <= 1.25 x SC-70 pad)

Co-Authored-By: Claude Opus 5.5 <noreply@anthropic.com>
Claude-Session: https://claude.ai/code/session_01YRUiF8Vp4242sya9Xyg3TV
Parts:
- removed R14, R15, R16, R17, R18, R19, R20: 10k, Resistor_SMD:R_0603_1608Metric, symbol Device:R
- removed TP2: SPARE_P14, TestPoint:TestPoint_Pad_D1.0mm, symbol Connector:TestPoint
- removed TP3: SPARE_P15, TestPoint:TestPoint_Pad_D1.0mm, symbol Connector:TestPoint
- removed TP4: SPARE_P16, TestPoint:TestPoint_Pad_D1.0mm, symbol Connector:TestPoint
- removed TP5: SPARE_P17, TestPoint:TestPoint_Pad_D1.0mm, symbol Connector:TestPoint
- removed TP7: 3V3, TestPoint:TestPoint_Pad_D1.0mm, symbol Connector:TestPoint
- added C11, C7: 100nF/16V/10%, Capacitor_SMD:C_0603_1608Metric, symbol Device:C
- added C2: 10nF/50V/10%, Capacitor_SMD:C_0603_1608Metric, symbol Device:C
- added R6: 100k/5%, Resistor_SMD:R_0603_1608Metric, symbol Device:R
- added R8: 1k/1%, Resistor_SMD:R_0603_1608Metric, symbol Device:R
- C14: value 1u -> 1uF/16V/10%
- C15: value 100n -> 100nF/16V/10%
- J1: value C2 -> C2_DEBUG
- R13: value 10k -> 10k/5%
- TP1: value TP_TX -> TP/TX
- TP6: value SENSE -> TP/SENSE; Zone DIGITAL -> ANALOG
- U5: value EFM8BB21F16G-C-QSOP24 -> EFM8BB21F16G-C(QSOP24); MPN EFM8BB21F16G-C-QSOP24 -> (none)
Connections:
- net +3V3: now also J1.4 (Pin_4), R6.1; no longer J1.1 (Pin_1)
- net FAULT_N: now also R6.2
- net GND: now also J1.1 (Pin_1), C11.2, C2.2, C7.2; no longer J1.4 (Pin_4)
- net ILNA: now also R8.1; no longer U5.1 (P0.3/EXTCLK)
- net SCAP_ADC: now also C11.1
- net SENSE: now also C2.1
- net C2D: no longer names the net of J1.2 (Pin_2), U5.8 (P3.0/C2D)
- net RST_N: no longer names the net of J1.3 (Pin_3), R13.2, U5.7 (RSTb/C2CK)
- net SPARE_P14: no longer names the net of U5.16 (P1.4)
- net SPARE_P15: no longer names the net of U5.15 (P1.5)
- net SPARE_P16: no longer names the net of U5.14 (P1.6)
- net SPARE_P17: no longer names the net of U5.13 (P1.7)
- net TP_TX: no longer names the net of TP1.1, U5.24 (P0.4/TX)
- new net: C7.1, R8.2, U5.1 (P0.3/ADC)
- no-connect marks 0 -> 4
Other:
- note added: "J1: 1=GND 2=C2D 3=C2CK 4=3V3"
- note added: "MCU"
- note added: "Pinout follows placement: QSOP pins 1-12 (ADC, debug, lamp chain P2.x) face power/panel,"
- note added: "SYSCLK = HFOSC0/8 = 3.0625 MHz, Snooze when idle (no clock, no spurs). ILNA RC: fc = 1.6 kHz"
- note added: "pins 13-24 (switch control, LNA_EN, FAULT_N) face the RF chain: no line crosses the MCU."
- note removed: "4-pin 2.54 mm: 3V3, C2D, C2CK(RSTb), GND. Works with a SiLabs debug adapter"
- note removed: "A EFM8BB21F16G-C-QSOP24"
- note removed: "B C2 debug / programming"
- note removed: "C Reset-safe defaults (pins are weak-pull-up / Hi-Z until firmware runs)"
- note removed: "D Test points"
- note removed: "OE_N pull-up keeps all lamps dark until the first panel write. FAULT_N pull-up is on the power sheet."
- note removed: "Pin map = firmware/src/hal_efm8bb2.c. P0.0 and P0.1 share SENSE (digital + ADC)."
- note removed: "Pins follow placement: QSOP pins 1-12 (analog, debug, lamp chain P2.x) face power/panel,"
- note removed: "Pull-downs: LNA off, bypass, branch 0 = THRU, FM notch out -> the box is a plain cable during reset."
- note removed: "SYSCLK HFOSC0/8 = 3.06 MHz; Snooze when idle (no clock -> no spurs). Keep under the can."
- note removed: "TP_TX: firmware drives it low; route UART0 TX here for debug prints if ever needed."
- note removed: "or an Arduino-based C2 programmer. Do not add a cap on RSTb (C2 clock)."
- note removed: "pins 13-24 (switch control, LNA_EN, FAULT_N) face the RF chain. No control line crosses the MCU."
