File: hardware/kicad/mcu.kicad_sch (KiCad schematic)
At the start: 12 parts, among them J1 C2_DEBUG, U5 EFM8BB21F16G-C(QSOP24)

Commit message: U7 on its own GPIO (P1.4 LNA_PATH_OUT)
The output SPDT gets its own control line (same polarity, 10k pull-down),
so the two switches can also be set independently later (e.g. LNA in
circuit on one side only for tests). Firmware drives both together;
179/179 host checks pass.

Co-Authored-By: Claude Opus 5.5 <noreply@anthropic.com>
Claude-Session: https://claude.ai/code/session_01YRUiF8Vp4242sya9Xyg3TV
Connections:
- net LNA_PATH_OUT: now reaches U5.16 (P1.4)
- no-connect marks 4 -> 3
Changed lines of the file:
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@@
     (instances
       (project "coaxolotl"
-        (path "/67534585-e0b7-41de-be56-14f8de14b6b9/fa9b5881-0f05-4368-a6d3-7b8504d3c635"
+        (path "/bb493d16-8963-485a-b4d1-cc07b45b8f8e/4aaebbfb-043b-40fa-b3f0-04c7e0b6523a"
           (reference "U5")
           (unit 1)
@@
     (instances
       (project "coaxolotl"
-        (path "/67534585-e0b7-41de-be56-14f8de14b6b9/fa9b5881-0f05-4368-a6d3-7b8504d3c635"
+        (path "/bb493d16-8963-485a-b4d1-cc07b45b8f8e/4aaebbfb-043b-40fa-b3f0-04c7e0b6523a"
           (reference "C15")
           (unit 1)
@@
     (instances
       (project "coaxolotl"
-        (path "/67534585-e0b7-41de-be56-14f8de14b6b9/fa9b5881-0f05-4368-a6d3-7b8504d3c635"
+        (path "/bb493d16-8963-485a-b4d1-cc07b45b8f8e/4aaebbfb-043b-40fa-b3f0-04c7e0b6523a"
           (reference "C14")
           (unit 1)
@@
     (instances
       (project "coaxolotl"
-        (path "/67534585-e0b7-41de-be56-14f8de14b6b9/fa9b5881-0f05-4368-a6d3-7b8504d3c635"
+        (path "/bb493d16-8963-485a-b4d1-cc07b45b8f8e/4aaebbfb-043b-40fa-b3f0-04c7e0b6523a"
           (reference "#PWR001")
           (unit 1)
@@
     (instances
       (project "coaxolotl"
-        (path "/67534585-e0b7-41de-be56-14f8de14b6b9/fa9b5881-0f05-4368-a6d3-7b8504d3c635"
+        (path "/bb493d16-8963-485a-b4d1-cc07b45b8f8e/4aaebbfb-043b-40fa-b3f0-04c7e0b6523a"
           (reference "#PWR002")
           (unit 1)
@@
     (instances
       (project "coaxolotl"
-        (path "/67534585-e0b7-41de-be56-14f8de14b6b9/fa9b5881-0f05-4368-a6d3-7b8504d3c635"
+        (path "/bb493d16-8963-485a-b4d1-cc07b45b8f8e/4aaebbfb-043b-40fa-b3f0-04c7e0b6523a"
           (reference "#PWR003")
           (unit 1)
@@
     (instances
       (project "coaxolotl"
-        (path "/67534585-e0b7-41de-be56-14f8de14b6b9/fa9b5881-0f05-4368-a6d3-7b8504d3c635"
+        (path "/bb493d16-8963-485a-b4d1-cc07b45b8f8e/4aaebbfb-043b-40fa-b3f0-04c7e0b6523a"
           (reference "#PWR004")
           (unit 1)
@@
     (instances
       (project "coaxolotl"
-        (path "/67534585-e0b7-41de-be56-14f8de14b6b9/fa9b5881-0f05-4368-a6d3-7b8504d3c635"
+        (path "/bb493d16-8963-485a-b4d1-cc07b45b8f8e/4aaebbfb-043b-40fa-b3f0-04c7e0b6523a"
           (reference "J1")
           (unit 1)
@@
     (instances
       (project "coaxolotl"
-        (path "/67534585-e0b7-41de-be56-14f8de14b6b9/fa9b5881-0f05-4368-a6d3-7b8504d3c635"
+        (path "/bb493d16-8963-485a-b4d1-cc07b45b8f8e/4aaebbfb-043b-40fa-b3f0-04c7e0b6523a"
           (reference "R13")
           (unit 1)
@@
     (instances
       (project "coaxolotl"
-        (path "/67534585-e0b7-41de-be56-14f8de14b6b9/fa9b5881-0f05-4368-a6d3-7b8504d3c635"
+        (path "/bb493d16-8963-485a-b4d1-cc07b45b8f8e/4aaebbfb-043b-40fa-b3f0-04c7e0b6523a"
           (reference "#PWR005")
           (unit 1)
@@
     (instances
       (project "coaxolotl"
-        (path "/67534585-e0b7-41de-be56-14f8de14b6b9/fa9b5881-0f05-4368-a6d3-7b8504d3c635"
+        (path "/bb493d16-8963-485a-b4d1-cc07b45b8f8e/4aaebbfb-043b-40fa-b3f0-04c7e0b6523a"
           (reference "#PWR006")
           (unit 1)
@@
     (instances
       (project "coaxolotl"
-        (path "/67534585-e0b7-41de-be56-14f8de14b6b9/fa9b5881-0f05-4368-a6d3-7b8504d3c635"
+        (path "/bb493d16-8963-485a-b4d1-cc07b45b8f8e/4aaebbfb-043b-40fa-b3f0-04c7e0b6523a"
           (reference "#PWR007")
           (unit 1)
@@
     (instances
       (project "coaxolotl"
-        (path "/67534585-e0b7-41de-be56-14f8de14b6b9/fa9b5881-0f05-4368-a6d3-7b8504d3c635"
+        (path "/bb493d16-8963-485a-b4d1-cc07b45b8f8e/4aaebbfb-043b-40fa-b3f0-04c7e0b6523a"
           (reference "R6")
           (unit 1)
@@
     (instances
       (project "coaxolotl"
-        (path "/67534585-e0b7-41de-be56-14f8de14b6b9/fa9b5881-0f05-4368-a6d3-7b8504d3c635"
+        (path "/bb493d16-8963-485a-b4d1-cc07b45b8f8e/4aaebbfb-043b-40fa-b3f0-04c7e0b6523a"
           (reference "#PWR008")
           (unit 1)
@@
     (instances
       (project "coaxolotl"
-        (path "/67534585-e0b7-41de-be56-14f8de14b6b9/fa9b5881-0f05-4368-a6d3-7b8504d3c635"
+        (path "/bb493d16-8963-485a-b4d1-cc07b45b8f8e/4aaebbfb-043b-40fa-b3f0-04c7e0b6523a"
           (reference "R8")
           (unit 1)
@@
     (instances
       (project "coaxolotl"
-        (path "/67534585-e0b7-41de-be56-14f8de14b6b9/fa9b5881-0f05-4368-a6d3-7b8504d3c635"
+        (path "/bb493d16-8963-485a-b4d1-cc07b45b8f8e/4aaebbfb-043b-40fa-b3f0-04c7e0b6523a"
           (reference "C7")
           (unit 1)
@@
     (instances
       (project "coaxolotl"
-        (path "/67534585-e0b7-41de-be56-14f8de14b6b9/fa9b5881-0f05-4368-a6d3-7b8504d3c635"
+        (path "/bb493d16-8963-485a-b4d1-cc07b45b8f8e/4aaebbfb-043b-40fa-b3f0-04c7e0b6523a"
           (reference "C11")
           (unit 1)
@@
     (instances
       (project "coaxolotl"
-        (path "/67534585-e0b7-41de-be56-14f8de14b6b9/fa9b5881-0f05-4368-a6d3-7b8504d3c635"
+        (path "/bb493d16-8963-485a-b4d1-cc07b45b8f8e/4aaebbfb-043b-40fa-b3f0-04c7e0b6523a"
           (reference "C2")
           (unit 1)
@@
     (instances
       (project "coaxolotl"
-        (path "/67534585-e0b7-41de-be56-14f8de14b6b9/fa9b5881-0f05-4368-a6d3-7b8504d3c635"
+        (path "/bb493d16-8963-485a-b4d1-cc07b45b8f8e/4aaebbfb-043b-40fa-b3f0-04c7e0b6523a"
           (reference "TP6")
           (unit 1)
@@
     (instances
       (project "coaxolotl"
-        (path "/67534585-e0b7-41de-be56-14f8de14b6b9/fa9b5881-0f05-4368-a6d3-7b8504d3c635"
+        (path "/bb493d16-8963-485a-b4d1-cc07b45b8f8e/4aaebbfb-043b-40fa-b3f0-04c7e0b6523a"
           (reference "TP1")
           (unit 1)
@@
     (instances
       (project "coaxolotl"
-        (path "/67534585-e0b7-41de-be56-14f8de14b6b9/fa9b5881-0f05-4368-a6d3-7b8504d3c635"
+        (path "/bb493d16-8963-485a-b4d1-cc07b45b8f8e/4aaebbfb-043b-40fa-b3f0-04c7e0b6523a"
           (reference "#PWR009")
           (unit 1)
@@
     (instances
       (project "coaxolotl"
-        (path "/67534585-e0b7-41de-be56-14f8de14b6b9/fa9b5881-0f05-4368-a6d3-7b8504d3c635"
+        (path "/bb493d16-8963-485a-b4d1-cc07b45b8f8e/4aaebbfb-043b-40fa-b3f0-04c7e0b6523a"
           (reference "#PWR010")
           (unit 1)
@@
     (instances
       (project "coaxolotl"
-        (path "/67534585-e0b7-41de-be56-14f8de14b6b9/fa9b5881-0f05-4368-a6d3-7b8504d3c635"
+        (path "/bb493d16-8963-485a-b4d1-cc07b45b8f8e/4aaebbfb-043b-40fa-b3f0-04c7e0b6523a"
           (reference "#PWR011")
           (unit 1)
@@
     )
   )
+  (hierarchical_label "LNA_PATH_OUT"
+    (shape output)
+    (at 215.9 114.3 0)
+    (fields_autoplaced)
+    (effects
+      (font
+        (face "Arial")
+        (size 1.27 1.27)
+      )
+      (justify left)
+    )
+  )
   (hierarchical_label "LED_SER"
     (shape output)
@@
   )
   (no_connect
-    (at 182.88 114.3)
-  )
-  (no_connect
     (at 182.88 116.84)
   )
@@
     )
     (stroke
+      (width 0)
+      (type default)
+    )
+  )
+  (wire
+    (pts
+      (xy 182.88 114.3)
+      (xy 215.9 114.3)
+    )
+    (stroke
