File: hardware/kicad/power.kicad_sch (KiCad schematic)
At the start: 35 parts, among them U1 LM66100DCKR, U2 TPS2553DBVR, U3 INA180A2IDBVR, U4 MCP1700T-3302E/TT

Commit message: WIP: zone/place fields, lamp chain moved to P2.0-P2.3, power sheet re-flow
Pin sides follow placement (QSOP pins 1-12 power/panel side, 13-24 RF side).
Block diagram and Olimex-style restyle still pending.

Co-Authored-By: Claude Opus 5.5 <noreply@anthropic.com>
Claude-Session: https://claude.ai/code/session_01YRUiF8Vp4242sya9Xyg3TV
Parts:
- C1: Place (none) -> D1; Zone (none) -> POWER
- C10, D2, D3, D4, D5, FB1, R1, R10, R2, R9, U1, U2, U4: Zone (none) -> POWER
- C11, R12: Place (none) -> U5.2; Zone (none) -> ANALOG
- C12: Place (none) -> U4.3; Zone (none) -> POWER
- C13: Place (none) -> U4.2; Zone (none) -> POWER
- C2: Place (none) -> U5.4 (SENSE at the MCU pin); Zone (none) -> ANALOG
- C3: Place (none) -> U1.6; Zone (none) -> POWER
- C4: Place (none) -> U2.1; Zone (none) -> POWER
- C5: Place (none) -> U2.6; Zone (none) -> POWER
- C6: Place (none) -> U3.5; Zone (none) -> ANALOG
- C7: Place (none) -> U5.1; Zone (none) -> ANALOG
- C8: Place (none) -> first 74HC595 (panel sheet); Zone (none) -> POWER
- C9: Place (none) -> D3 cathode / U4.3; Zone (none) -> POWER
- D1: Place (none) -> edge:J_COAX (RF sheet bias-T), shortest GND return; Zone (none) -> POWER
- R11: Place (none) -> C10; Zone (none) -> ANALOG
- R3: Place (none) -> VCOAX tap; Zone (none) -> ANALOG
- R4: Place (none) -> R3; Zone (none) -> ANALOG
- R5: Place (none) -> U2.5 (short ILIM loop); Zone (none) -> POWER
- R6: Place (none) -> U2.4; Zone (none) -> POWER
- R7: Place (none) -> between U2.6 and LNA feed; Zone (none) -> POWER
- R8: Place (none) -> U5.1 (ILNA RC at the ADC pin); Zone (none) -> ANALOG
- U3: Zone (none) -> ANALOG

Commit message: Schematic v0.2: Olimex-style redraw with block diagram
- power/ground only as power symbols (project rails VCOAX, VMAIN, VHOLD, VLED, LNA_VCC)
- wires inside blocks, hierarchical labels + sheet pins between sheets (no global labels)
- Value carries critical parameters, blue design-intent notes, bold italic block titles
- sheet 1: block diagram + wired hierarchy; RF/Panel placeholders with reset-safe pulls
- pull-downs moved to the receiving parts (TPS2553 EN, RF switches), RC filters to the ADC pins
- check.py compares net partitions (catches shorts and splits), generator flags 4-way junctions
- net classes in .kicad_pro (POWER 0.4 mm <= 1.25 x SC-70 pad)

Co-Authored-By: Claude Opus 5.5 <noreply@anthropic.com>
Claude-Session: https://claude.ai/code/session_01YRUiF8Vp4242sya9Xyg3TV
Parts:
- removed C11, C7: 100n, Capacitor_SMD:C_0603_1608Metric, symbol Device:C
- removed C2: 10n, Capacitor_SMD:C_0603_1608Metric, symbol Device:C
- removed R6: 100k, Resistor_SMD:R_0603_1608Metric, symbol Device:R
- removed R8: 1k, Resistor_SMD:R_0603_1608Metric, symbol Device:R
- removed U3: INA180A2IDBVR, Package_TO_SOT_SMD:SOT-23-5, symbol Amplifier_Current:INA180A2
- added R14: 10k/5%, Resistor_SMD:R_0603_1608Metric, symbol Device:R
- added U3: INA180A2IDBVR(SOT23-5), Package_TO_SOT_SMD:SOT-23-5, symbol coaxolotl:INA180A2
- C1: value 100n -> 100nF/16V/10%; Place D1 -> (none)
- C10: value 0.1F 5.5V -> 0.1F/5.5V
- C12, C13, C4, C5: value 1u -> 1uF/16V/10%
- C3: value 10u 10V -> 10uF/10V/20%
- C6: value 100n -> 100nF/16V/10%
- C8: value 47u 10V -> 47uF/10V/20%; Place first 74HC595 (panel sheet) -> (none)
- C9: value 330u 6.3V polymer -> 330uF/6.3V/20%; Place D3 cathode / U4.3 -> (none)
- D1: value SMF5.0A -> SMF5.0A(SOD123F); MPN SMF5.0A -> (none); Place edge:J_COAX (RF sheet bias-T), shortest GND return -> at J_COAX (RF sheet)
- D2: value PWR green -> LED/GREEN(0603); Note (none) -> PWR lamp, works without MCU
- D3, D4, D5: value BAT54WS -> BAT54WS(SOD323); MPN BAT54WS -> (none)
- FB1: value 600R@100MHz -> FB0603/600R/1.3A
- R1: value 680 -> 680R/1%; Note (none) -> sets the OOK falling edge
- R10: value 220 -> 220R/5%
- R11: value 1M -> 1M/1%; Place C10 -> (none)
- R12: value 1M -> 1M/1%; Place U5.2 -> (none)
- R2: value 3k3 -> 3k3/5%
- R3: value 10k 1% -> 10k/1%; Place VCOAX tap -> (none)
- R4: value 22k 1% -> 22k/1%; Place R3 -> (none)
- R5: value 150k 1% -> 150k/1%; Note VERIFY vs TPS2553 Eq.1 -> VERIFY vs TPS2553 Eq.1: IOS(min) > 130 mA; Place U2.5 (short ILIM loop) -> U2.5
- R7: value 0R39 1% -> 0R39/1%/0.25W; Place between U2.6 and LNA feed -> (none)
- R9: value 100 -> 100R/5%
- U1: value LM66100DCKR -> LM66100DCKR(SC70-6); MPN LM66100DCKR -> (none)
- U2: value TPS2553DBVR -> TPS2553DBVR(SOT23-6); MPN TPS2553DBVR -> (none)
- U4: value MCP1700T-3302E/TT -> MCP1700T-3302E/TT(SOT23); MPN MCP1700T-3302E/TT -> (none)
Connections:
- net +3V3: now also U3.5 (V+)
- net GND: now also R14.2, U3.2 (GND)
- net ILNA: now also U3.1 (OUT)
- net LNA_EN: now also R14.1
- net LNA_VCC: now also U3.4 (IN-)
- net HU_FAST: no longer names the net of D3.2 (A), R9.2
- net ILIM: no longer names the net of R5.1, U2.5 (ILIM)
- net LNA_SW: no longer names the net of C5.1, R7.1, U2.6 (OUT)
- net LNA_SW: now also U3.3 (IN+)
- net PWR_LED_A: no longer names the net of D2.2 (A), R2.2
- net SC_CHG: no longer names the net of D4.2 (A), R10.2
- net VSCAP: no longer names the net of C10.1, D4.1 (K), D5.2 (A), R11.1
Other:
- note added: "3V3 regulator"
- note added: "48 lamps x 1 mA max on VMAIN:"
- note added: "CE = VOUT: comparator blocks"
- note added: "Hold-up (diode-OR)"
- note added: "ILNA = 0.39R x 50 V/V = 19.5 mV/mA (100 mA -> 1.95 V); Kelvin taps at R7 pads"
- note added: "Ideal diode"
- note added: "Ilim = f(R5), TPS2553 Eq.1: VERIFY IOS(min) > 130 mA"
- note added: "LNA supply + current monitor"
- note added: "Lamp rail"
- note added: "MCP1700: Iq 1.6 uA, dropout 178 mV;"
- note added: "SCAP_ADC = VSCAP / 2 (HOLD lamp at >= 3.6 V)"
- note added: "SENSE = 0.6875 x VCOAX (3.0 V at 4.4 V)"
- note added: "VCOAX tap"
- note added: "VO needs >= 1 uF ceramic"
- note added: "dark in OOK gaps, no hold-up drain"
- note added: "fast path R9/D3: VHOLD up in ~30 ms (100R x 330uF) -> MCU boots"
- note added: "reverse current in OOK gaps"
- note added: "slow path R10/D4: tau ~22 s (220R x 0.1F); ride-through ~4 min at 0.6 mA"
- note added: "t_fall = 1.1 x R_eff x C_total: R1 sets the OOK falling edge"
- note removed: "(<=18 mA, tau ~22 s). D5 lets the supercap carry VHOLD through a dropout (~4 min @ 0.6 mA)."
- note removed: "A VCOAX tap (ahead of all bulk capacitance)"
- note removed: "B Ideal diode VCOAX -> VMAIN"
- note removed: "C LNA supply: current-limited switch + shunt monitor"
- note removed: "CE tied to VOUT: the comparator turns the FET off whenever VMAIN > VCOAX,"
- note removed: "D Lamp rail"
- note removed: "E Hold-up: fast 330 uF + 0.1 F supercap, diode-OR"
- note removed: "F 3V3 for MCU, switches, INA180, 595s"
- note removed: "Fast path R9/D3 boots the MCU in ~30 ms. Slow path R10/D4 charges the supercap"
- note removed: "LNA_VCC continues to the LNA bias filter on the RF sheet."
- note removed: "Lamps hang on VMAIN (not the hold-up): they go dark in every OOK gap"
- note removed: "MCP1700: 1.6 uA Iq, 178 mV dropout. Needs >= 1 uF ceramic on the output."
- note removed: "Only these loads sit on VCOAX, so the OOK falling edge is set by R1 + coax/RTL capacitance."
- note removed: "R1 = 680R gives ~6 ms with 10 uF on the RTL side; lower to 470R if bring-up step 1 needs it."
- note removed: "R5 VERIFY: pick from datasheet Eq.1 / Fig.22 for IOS(min) > 130 mA (1% part)."
- note removed: "SCAP_ADC = VSCAP / 2 -> P0.2 (HOLD lamp)."
- note removed: "SENSE = 0.69 x VCOAX (3.0 V @ 4.4 V). Goes to P0.0 (port match) and P0.1 (ADC)."
- note removed: "ST unused -> GND (datasheet)."
- note removed: "Shunt 0.39R x INA180A2 (50 V/V) = 19.5 mV/mA -> 100 mA = 1.95 V at P0.3."
- note removed: "TPS2553: EN active-high, 8 ms FAULT deglitch, ILIM tied to IN = 75 mA typ (too low)."
- note removed: "and in a dropout instead of draining the supercap. 48 x ~1 mA max."
- note removed: "so LNA, lamps and hold-up never back-feed the sense node during a gap."
