File: hardware/kicad/power.kicad_sch (KiCad schematic)
At the start: 31 parts, among them U1 LM66100DCKR(SC70-6), U2 TPS2553DBVR(SOT23-6), U3 INA180A2IDBVR(SOT23-5), U4 MCP1700T-3302E/TT(SOT23)

Commit message: Filter bank F7 retuned for the pad capacitance; LCSC codes for every fitted part; C10/J1/TP1/TP6 DNP
F7 (70/23cm HPF): C701/C703 12 pF, C702 6.8 pF, L701/L702 10 nH (was 8.2p/4.7p/15n), from the
openEMS lane N-port co-simulation (simu/f7_retune.py). filters.LAYOUT_TUNED carries the values.
L403/L404: Murata LQW18ANR33G00D C162651 (ceramic core) replaces LQW18CAR33J00D.
New codes, checked on JLC/LCSC (EasyEDA API) 2026-10-28: 12pF C38523, 6.8pF C1679, 10nH C15666,
820pF C701305, 1.5uH C317997, 2.2uH C41651, 4.7uH C139136.
Schematic sheets patched in place (build.py writes random uuids; the routed board links to the
current ones); build.py carries the same changes.

Co-Authored-By: Claude Opus 5.5 <noreply@anthropic.com>
Claude-Session: https://claude.ai/code/session_01YRUiF8Vp4242sya9Xyg3TV
Parts:
- C10: Note VERIFY footprint vs chosen coin supercap -> VERIFY footprint vs chosen coin supercap; hand-soldered (no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; now not fitted
Changed lines of the file:
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@@
     (in_bom yes)
     (on_board yes)
-    (dnp no)
+    (dnp yes)
     (property "Reference" "C10"
       (at 78.74 154.94 0)
@@
       )
     )
-    (property "Note" "VERIFY footprint vs chosen coin supercap"
+    (property "Note" "VERIFY footprint vs chosen coin supercap; hand-soldered (no LCSC part)"
       (at 80.01 156.21 0)
       (effects
