File: hardware/kicad/filterbank.kicad_sch (KiCad schematic)
At the start: 23 parts, among them J3 SMA/EDGE(RTL-SDR), U11 PE42582A(QFN24), U8 PE42582A(QFN24)

Commit message: Schematic: real F1-F7 LC filters, snap-off lamp strip link
- tools/filters.py: 5th-order Chebyshev 0.1 dB ladders, 50 ohm, E12;
  BPF = HPF + LPF; prints the rounded-value response. F5 is now 30-80 MHz
  (12 dB at 98 MHz instead of 1 dB), bandplan.json updated.
- Filter bank sheet redrawn around the ladders (C1xx..C7xx, L1xx..L7xx).
- Panel sheet: J4/J5 unpopulated 1x7 rows at the right end of the break
  line, so a snapped-off lamp strip can be re-linked with a cable.
- BOM regenerated (224 parts).

Co-Authored-By: Claude Opus 5.5 <noreply@anthropic.com>
Claude-Session: https://claude.ai/code/session_01YRUiF8Vp4242sya9Xyg3TV
Parts:
- removed FL1: F1 LPF 550 kHz, coaxolotl:FILTER_TBD, symbol coaxolotl:RF_FILTER
- removed FL2: F2 BPF 1.6-4 MHz, coaxolotl:FILTER_TBD, symbol coaxolotl:RF_FILTER
- removed FL3: F3 BPF 4-12 MHz, coaxolotl:FILTER_TBD, symbol coaxolotl:RF_FILTER
- removed FL4: F4 BPF 12-30 MHz, coaxolotl:FILTER_TBD, symbol coaxolotl:RF_FILTER
- removed FL5: F5 BPF 30-88 MHz, coaxolotl:FILTER_TBD, symbol coaxolotl:RF_FILTER
- removed FL6: F6 BPF 108-174 MHz, coaxolotl:FILTER_TBD, symbol coaxolotl:RF_FILTER
- removed FL7: F7 HPF 380 MHz, coaxolotl:FILTER_TBD, symbol coaxolotl:RF_FILTER
- added C101, C103: 5.6nF/50V/C0G, Capacitor_SMD:C_0603_1608Metric, symbol Device:C
- added C102: 10nF/50V/C0G, Capacitor_SMD:C_0603_1608Metric, symbol Device:C
- added C201, C203: 2.2nF/50V/C0G, Capacitor_SMD:C_0603_1608Metric, symbol Device:C
- added C202: 1.2nF/50V/C0G, Capacitor_SMD:C_0603_1608Metric, symbol Device:C
- added C204, C206, C301, C303: 820pF/50V/C0G, Capacitor_SMD:C_0603_1608Metric, symbol Device:C
- added C205: 1.5nF/50V/C0G, Capacitor_SMD:C_0603_1608Metric, symbol Device:C
- added C302, C305: 470pF/50V/C0G, Capacitor_SMD:C_0603_1608Metric, symbol Device:C
- added C304, C306, C401, C403: 270pF/50V/C0G, Capacitor_SMD:C_0603_1608Metric, symbol Device:C
- added C402: 150pF/50V/C0G, Capacitor_SMD:C_0603_1608Metric, symbol Device:C
- added C404, C406, C501, C503: 100pF/50V/C0G, Capacitor_SMD:C_0603_1608Metric, symbol Device:C
- added C405: 180pF/50V/C0G, Capacitor_SMD:C_0603_1608Metric, symbol Device:C
- added C502: 56pF/50V/C0G, Capacitor_SMD:C_0603_1608Metric, symbol Device:C
- added C504, C506: 47pF/50V/C0G, Capacitor_SMD:C_0603_1608Metric, symbol Device:C
- added C505: 82pF/50V/C0G, Capacitor_SMD:C_0603_1608Metric, symbol Device:C
- added C601, C603: 27pF/50V/C0G, Capacitor_SMD:C_0603_1608Metric, symbol Device:C
- added C602: 15pF/50V/C0G, Capacitor_SMD:C_0603_1608Metric, symbol Device:C
- added C604, C606: 18pF/50V/C0G, Capacitor_SMD:C_0603_1608Metric, symbol Device:C
- added C605: 33pF/50V/C0G, Capacitor_SMD:C_0603_1608Metric, symbol Device:C
- added C701, C703: 8.2pF/50V/C0G, Capacitor_SMD:C_0603_1608Metric, symbol Device:C
- added C702: 4.7pF/50V/C0G, Capacitor_SMD:C_0603_1608Metric, symbol Device:C
- added L101, L102: 18uH/5%, Inductor_SMD:L_1210_3225Metric, symbol Device:L
- added L201, L202: 4.7uH/5%, Inductor_SMD:L_0805_2012Metric, symbol Device:L
- added L203, L204: 2.2uH/5%, Inductor_SMD:L_0805_2012Metric, symbol Device:L
- added L301, L302: 1.5uH/5%, Inductor_SMD:L_0805_2012Metric, symbol Device:L
- added L303, L304: 820nH/5%, Inductor_SMD:L_0805_2012Metric, symbol Device:L
- added L401, L402: 560nH/5%, Inductor_SMD:L_0805_2012Metric, symbol Device:L
- added L403, L404: 330nH/5%, Inductor_SMD:L_0603_1608Metric, symbol Device:L
- added L501, L502: 220nH/5%, Inductor_SMD:L_0603_1608Metric, symbol Device:L
- added L503, L504: 150nH/5%, Inductor_SMD:L_0603_1608Metric, symbol Device:L
- added L601, L602, L603, L604: 56nH/5%, Inductor_SMD:L_0603_1608Metric, symbol Device:L
- added L701, L702: 15nH/5%, Inductor_SMD:L_0603_1608Metric, symbol Device:L
Connections:
- net GND: now also C101.2, C102.2, C103.2, C204.2, C205.2, C206.2, C304.2, C305.2, C306.2, C404.2, C405.2, C406.2, C504.2, C505.2, C506.2, C604.2, C605.2, C606.2, L201.2, L202.2, L301.2, L302.2, L401.2, L402.2, L501.2, L502.2, L601.2, L602.2, L701.2, L702.2
- net at U8.13 (RF5): now also C401.1
- net at U11.13 (RF5): now also C406.1, L404.2
- net at U8.15 (RF6): now also C501.1
- net at U11.15 (RF6): now also C506.1, L504.2
- net at U8.2 (RF2): now also C101.1, L101.1
- net at U11.2 (RF2): now also C103.1, L102.2
- net at U8.17 (RF7): now also C601.1
- net at U11.17 (RF7): now also C606.1, L604.2
- net at U8.6 (RF4): now also C301.1
- net at U11.6 (RF4): now also C306.1, L304.2
- net at U8.19 (RF8): now also C701.1
- net at U8.4 (RF3): now also C201.1
- net at U11.19 (RF8): now also C703.2
- net at U11.4 (RF3): now also C206.1, L204.2
- new net: C102.1, L101.2, L102.1
- new net: C301.2, C302.1, L301.1
- new net: C203.2, C204.1, L203.1
- new net: C205.1, L203.2, L204.1
- new net: C503.2, C504.1, L503.1
- new net: C505.1, L503.2, L504.1
- new net: C701.2, C702.1, L701.1
- new net: C702.2, C703.1, L702.1
- new net: C201.2, C202.1, L201.1
- new net: C501.2, C502.1, L501.1
- new net: C602.2, C603.1, L602.1
- new net: C603.2, C604.1, L603.1
- new net: C605.1, L603.2, L604.1
- new net: C303.2, C304.1, L303.1
- new net: C305.1, L303.2, L304.1
- new net: C601.2, C602.1, L601.1
- new net: C401.2, C402.1, L401.1
- new net: C502.2, C503.1, L502.1
- new net: C202.2, C203.1, L202.1
- new net: C403.2, C404.1, L403.1
- new net: C405.1, L403.2, L404.1
- new net: C402.2, C403.1, L402.1
- new net: C302.2, C303.1, L302.1
Other:
- note added: "(mapped in tools/gen_bandplan.py). V4 = LS = VSS_EXT = GND."
- note added: "BPF = HPF + LPF (tools/filters.py). Ideal-part response there;"
- note added: "Branch k on RFk+1 of both switches. LS = 0 code (V3 V2 V1):"
- note added: "F1 LPF 550 kHz"
- note added: "F2 BPF 1.6-4 MHz"
- note added: "F3 BPF 4-12 MHz"
- note added: "F4 BPF 12-30 MHz"
- note added: "F5 BPF 30-80 MHz"
- note added: "F6 BPF 108-174 MHz"
- note added: "F7 HPF 380 MHz"
- note added: "Filters: 5th-order Chebyshev 0.1 dB, 50 ohm, E12 values,"
- note added: "RF1 000, RF2 100, RF3 010, RF4 110, RF5 001, RF6 101, RF7 011, RF8 111"
- note added: "VERIFY with real L Q / SRF and the layout on a VNA."
- note removed: "Branch k on RFk+1 of both switches. LS = 0 code (V3 V2 V1) per RF port: RF1 000, RF2 100, RF3 010, RF4 110, RF5 001, RF6 101, RF7 011, RF8 111"
- note removed: "Reset: V = 000 -> RF1 = F0 THRU (straight through)."
- note removed: "bandplan.json 'port' -> code mapping is done in tools/gen_bandplan.py. V4 = LS = VSS_EXT = GND (all-off unused, internal negative generator)."
