File: hardware/kicad/filterbank.kicad_sch (KiCad schematic)
At the start: 76 parts, among them J3 SMA/EDGE(RTL-SDR), U11 PE42582A(QFN24), U8 PE42582A(QFN24)

Commit message: J2/J3: BWSMA-KE-P001 air launch (z2labs DoE v14 coupon A0)
Through-milled notch 2.80 x 1.90 mm open to the board edge under the free pin (Edge.Cuts in the
footprint, the outline leaves the notch mouth open), signal pad 1.55 x 0.90 mm from the notch
bottom with 0.5 mm clearance (coplanar gap), leg pads 4.6 x 1.3 mm on F.Cu and B.Cu, launch via
pair 0.6/0.3 at (0.6, +-1.65). Origin on the board edge, J2 at x = 0, J3 at x = W rotated 180.
Pours keep the 0.3 mm board-edge clearance from the milled walls on every layer.

Co-Authored-By: Claude Opus 5.5 <noreply@anthropic.com>
Claude-Session: https://claude.ai/code/session_01YRUiF8Vp4242sya9Xyg3TV
Parts:
- J3: footprint coaxolotl:SMA_EdgeLaunch_BWSMA-KE-P001 -> coaxolotl:SMA_EdgeLaunch_BWSMA-KE-P001_Air
