File: hardware/kicad/panel.kicad_sch (KiCad schematic)
At the start: 75 parts, among them J4 NA(HDR1x7/2.54), J5 NA(HDR1x7/2.54), U14 74HC595PW(TSSOP16), U15 74HC595PW(TSSOP16), U16 74HC595PW(TSSOP16), U17 74HC595PW(TSSOP16), U18 74HC595PW(TSSOP16), U19 74HC595PW(TSSOP16)

Commit message: Lamp strip: each register drives the 4 columns above it (both rows), local wiring
Lamp n sits in row n/24, column n%24; register k drives columns 4k..4k+3 (QA-QD row 1, QE-QH row 2).
Schematic, netlist, hal_panel() shift order and docs/panel.md follow. Firmware tests 179/179.

Co-Authored-By: Claude Opus 5.5 <noreply@anthropic.com>
Claude-Session: https://claude.ai/code/session_01YRUiF8Vp4242sya9Xyg3TV
Connections:
- net at RN7.6 (R3.2): now also D21.1 (K); no longer D33.1 (K)
- net at D31.1 (K): now also RN2.8 (R1.2); no longer RN7.8 (R1.2)
- net at D24.1 (K): now also RN9.7 (R2.2); no longer RN5.7 (R2.2)
- net at RN9.8 (R1.2): now also D23.1 (K); no longer D39.1 (K)
- net at RN4.5 (R4.2): now also D38.1 (K); no longer D22.1 (K)
- net at RN9.6 (R3.2): now also D25.1 (K); no longer D41.1 (K)
- net at RN4.6 (R3.2): now also D37.1 (K); no longer D21.1 (K)
- net at RN3.5 (R4.2): now also D14.1 (K); no longer D18.1 (K)
- net at D12.1 (K): now also RN3.7 (R2.2); no longer RN2.7 (R2.2)
- net at RN2.5 (R4.2): now also D34.1 (K); no longer D14.1 (K)
- net at RN7.5 (R4.2): now also D22.1 (K); no longer D34.1 (K)
- net at D35.1 (K): now also RN4.8 (R1.2); no longer RN8.8 (R1.2)
- net at D26.1 (K): now also RN9.5 (R4.2); no longer RN5.5 (R4.2)
- net at RN5.6 (R3.2): now also D17.1 (K); no longer D25.1 (K)
- net at RN5.8 (R1.2): now also D15.1 (K); no longer D23.1 (K)
- net at RN4.7 (R2.2): now also D36.1 (K); no longer D20.1 (K)
- net at D19.1 (K): now also RN7.8 (R1.2); no longer RN4.8 (R1.2)
- net at D47.1 (K): now also RN10.8 (R1.2); no longer RN11.8 (R1.2)
- net at RN3.8 (R1.2): now also D11.1 (K); no longer D15.1 (K)
- net at D13.1 (K): now also RN3.6 (R3.2); no longer RN2.6 (R3.2)
- net at D27.1 (K): now also RN11.8 (R1.2); no longer RN6.8 (R1.2)
- net at D43.1 (K): now also RN8.8 (R1.2); no longer RN10.8 (R1.2)
- net at D16.1 (K): now also RN5.7 (R2.2); no longer RN3.7 (R2.2)
- net at D48.1 (K): now also RN10.7 (R2.2); no longer RN11.7 (R2.2)
- net at RN8.5 (R4.2): now also D46.1 (K); no longer D38.1 (K)
- net at D40.1 (K): now also RN6.7 (R2.2); no longer RN9.7 (R2.2)
- net at D28.1 (K): now also RN11.7 (R2.2); no longer RN6.7 (R2.2)
- net at D49.1 (K): now also RN10.6 (R3.2); no longer RN11.6 (R3.2)
- net at D29.1 (K): now also RN11.6 (R3.2); no longer RN6.6 (R3.2)
- net at RN10.5 (R4.2): now also D50.1 (K); no longer D46.1 (K)
- net at D30.1 (K): now also RN11.5 (R4.2); no longer RN6.5 (R4.2)
- net at D42.1 (K): now also RN6.5 (R4.2); no longer RN9.5 (R4.2)
- net at D45.1 (K): now also RN8.6 (R3.2); no longer RN10.6 (R3.2)
- net at D44.1 (K): now also RN8.7 (R2.2); no longer RN10.7 (R2.2)
- net at RN7.7 (R2.2): now also D20.1 (K); no longer D32.1 (K)
- new net: D41.1 (K), RN6.6 (R3.2)
- new net: D39.1 (K), RN6.8 (R1.2)
- new net: D33.1 (K), RN2.6 (R3.2)
- new net: D32.1 (K), RN2.7 (R2.2)
- new net: D18.1 (K), RN5.5 (R4.2)
Other:
- note added: "Lamp n: row n/24, column n%24; register (n%24)/4 (U14 first), output (n%4) + 4*(n/24) - hal_panel."
- note added: "Panel modes (config frame, kept in flash): full / bands = F0-F7 only / off = OE_N high."
- note added: "columns 0-3 (lamps 0-3, 24-27)"
- note added: "columns 12-15 (lamps 12-15, 36-39)"
- note added: "columns 16-19 (lamps 16-19, 40-43)"
- note added: "columns 20-23 (lamps 20-23, 44-47)"
- note added: "columns 4-7 (lamps 4-7, 28-31)"
- note added: "columns 8-11 (lamps 8-11, 32-35)"
- note removed: "BANK (lamps 0-7)"
- note removed: "DECODE (lamps 24-31)"
- note removed: "DECODE + RF (lamps 32-39)"
- note removed: "FRAME (lamps 8-15)"
- note removed: "FRAME + RX (lamps 16-23)"
- note removed: "Lamp n: register n/8 (U14 = first after the MCU), output Q(n%8) - firmware/src/panel.h."
- note removed: "Panel modes (config frame, kept in flash): full / bands = U14 only / off = OE_N high."
- note removed: "RF + SYSTEM (lamps 40-47)"
