File: hardware/kicad/rf_frontend.kicad_sch (KiCad schematic)
At the start: 31 parts, among them J2 SMA/EDGE(ANT), U10 NA(PE42520C-Z), U12 LFCN-2250+(FV1206), U13 QPL9547TR7(DFN8-2x2), U6 PE42520C-Z(QFN16), U7 PE42520C-Z(QFN16), U9 NA(PE42520C-Z)

Commit message: Project footprints: GDT 1812 (SANTE 4532-090V, C476204), FV1206 LTCC filter
Pads from the LCSC/EasyEDA footprints so JLC's own placement fits.

Co-Authored-By: Claude Opus 5.5 <noreply@anthropic.com>
Claude-Session: https://claude.ai/code/session_01YRUiF8Vp4242sya9Xyg3TV
Parts:
- GDT1: value GDT/90V -> 4532-090V(1812); footprint coaxolotl:GDT_SMD_VERIFY -> coaxolotl:GDT_SMD_1812; LCSC (none) -> C476204; MPN 2027-09-SM-RPLF -> 4532-090V; Note (none) -> 90 V, 0.5 pF

Commit message: U7/U10 with LS = GND (RF ports swapped) so the LNA/bypass ring is planar
Two identical SPDTs facing each other need one path to cross on a single
layer. With LS tied to GND on the output switch (and on the notch output)
CTRL = 0 selects RF2, so bypass goes RF1 -> RF2 and the LNA path RF2 ->
RF1: no crossing, no firmware change. Symbol variant PE42520R.

Co-Authored-By: Claude Opus 5.5 <noreply@anthropic.com>
Claude-Session: https://claude.ai/code/session_01YRUiF8Vp4242sya9Xyg3TV
Parts:
- removed U10: NA(PE42520C-Z), Package_DFN_QFN:QFN-16-1EP_3x3mm_P0.5mm_EP1.7x1.7mm, symbol coaxolotl:PE42520
- removed U7: PE42520C-Z(QFN16), Package_DFN_QFN:QFN-16-1EP_3x3mm_P0.5mm_EP1.7x1.7mm, symbol coaxolotl:PE42520
- added U10: NA(PE42520C-Z), Package_DFN_QFN:QFN-16-1EP_3x3mm_P0.5mm_EP1.7x1.7mm, symbol coaxolotl:PE42520R
- added U7: PE42520C-Z(QFN16), Package_DFN_QFN:QFN-16-1EP_3x3mm_P0.5mm_EP1.7x1.7mm, symbol coaxolotl:PE42520R
Connections:
- net +3V3: now also U10.16 (VDD), U7.16 (VDD)
- net FMN: now also U10.14 (CTRL)
- net GND: now also U10.1 (GND), U10.10 (GND), U10.12 (GND), U10.13 (GND), U10.15 (LS), U10.17 (GND), U10.3 (GND), U10.4 (GND), U10.5 (GND), U10.6 (GND), U10.8 (GND), U10.9 (GND), U7.1 (GND), U7.10 (GND), U7.12 (GND), U7.13 (GND), U7.15 (LS), U7.17 (GND), U7.3 (GND), U7.4 (GND), U7.5 (GND), U7.6 (GND), U7.8 (GND), U7.9 (GND)
- net LNA_PATH: now also U7.14 (CTRL)
- net RF_BANK: now also U7.7 (RFC)
- net at C27.2, L3.2: now also U10.2 (RF1)
- net at C28.1, R22.2: now also U10.7 (RFC)
- net at U9.2 (RF1): now also U10.11 (RF2)
- net at U6.2 (RF1): now also U7.11 (RF2)
- net at C31.2: now also U7.2 (RF1)
Other:
- note added: "LNA_PATH 0 = bypass, 1 = LNA; FMN 0 = through. U7/U10 have LS = GND (RF ports swapped: one-layer ring)."
- note removed: "LNA_PATH: 0 = RF1 = bypass, 1 = RF2 = LNA. FMN: 0 = RF1 = through, 1 = RF2 = notch."

Commit message: U7 on its own GPIO (P1.4 LNA_PATH_OUT)
The output SPDT gets its own control line (same polarity, 10k pull-down),
so the two switches can also be set independently later (e.g. LNA in
circuit on one side only for tests). Firmware drives both together;
179/179 host checks pass.

Co-Authored-By: Claude Opus 5.5 <noreply@anthropic.com>
Claude-Session: https://claude.ai/code/session_01YRUiF8Vp4242sya9Xyg3TV
Parts:
- added R26: 10k/5%, Resistor_SMD:R_0603_1608Metric, symbol Device:R
Connections:
- net GND: now also R26.2
- net LNA_PATH: no longer U7.14 (CTRL)
- new net LNA_PATH_OUT: R26.1, U7.14 (CTRL)
Other:
- note added: "LNA_PATH (U6) and LNA_PATH_OUT (U7, own GPIO): 0 = bypass, 1 = LNA. FMN 0 = through. U7/U10: LS = GND."
- note removed: "LNA_PATH 0 = bypass, 1 = LNA; FMN 0 = through. U7/U10 have LS = GND (RF ports swapped: one-layer ring)."

Commit message: MCU to EFM8BB21F16G-C-QFN20 (QSOP24 end of life), BWSMA-KE-P001 edge SMA, Brightking GDT
U5: QFN20, all 16 port pins used. TP_TX test point dropped; LED_OE_N on P0.4, lamp chain on
P1.4-P1.6, LNA_PATH_OUT on P1.3, FMN on P2.0/C2D through R30 1k (debugger overrides it).
Footprint from the LCSC C80713 land pattern. Firmware HAL and docs/hardware.md follow;
179/179 host tests pass, SDCC build OK.
J2/J3: BAT WIRELESS BWSMA-KE-P001 (C496550) edge launch, footprint from LCSC, board edge at
local x = +2.70 mm. GDT1: Brightking 4532-091-LF (C78323), same 1812 land pattern.
check.py: netlist matches the intent.

Co-Authored-By: Claude Opus 5.5 <noreply@anthropic.com>
Claude-Session: https://claude.ai/code/session_01YRUiF8Vp4242sya9Xyg3TV
Parts:
- C27: dnp yes -> (none); now not fitted
- GDT1: value 4532-090V(1812) -> 4532-091-LF(1812); LCSC C476204 -> C78323; MPN 4532-090V -> 4532-091-LF; Note 90 V, 0.5 pF -> 90 V, Brightking 4532 series
- J2: footprint Connector_Coaxial:SMA_Amphenol_132289_EdgeMount -> coaxolotl:SMA_EdgeLaunch_BWSMA-KE-P001

Commit message: J2/J3: BWSMA-KE-P001 air launch (z2labs DoE v14 coupon A0)
Through-milled notch 2.80 x 1.90 mm open to the board edge under the free pin (Edge.Cuts in the
footprint, the outline leaves the notch mouth open), signal pad 1.55 x 0.90 mm from the notch
bottom with 0.5 mm clearance (coplanar gap), leg pads 4.6 x 1.3 mm on F.Cu and B.Cu, launch via
pair 0.6/0.3 at (0.6, +-1.65). Origin on the board edge, J2 at x = 0, J3 at x = W rotated 180.
Pours keep the 0.3 mm board-edge clearance from the milled walls on every layer.

Co-Authored-By: Claude Opus 5.5 <noreply@anthropic.com>
Claude-Session: https://claude.ai/code/session_01YRUiF8Vp4242sya9Xyg3TV
Parts:
- J2: footprint coaxolotl:SMA_EdgeLaunch_BWSMA-KE-P001 -> coaxolotl:SMA_EdgeLaunch_BWSMA-KE-P001_Air
