File: hardware/kicad/coaxolotl_placed.kicad_pcb (KiCad board)
At the start: 4 copper layers, 100 x 102 mm, 243 parts, among them J1 C2_DEBUG, J2 SMA/EDGE(ANT), J3 SMA/EDGE(RTL-SDR), J4 NA(HDR1x7/2.54), J5 NA(HDR1x7/2.54), U1 LM66100DCKR(SC70-6), U10 NA(PE42520C-Z), U11 PE42582A(QFN24), U12 LFCN-2250+(FV1206), U13 QPL9547TR7(DFN8-2x2), U14 74HC595PW(TSSOP16), U15 74HC595PW(TSSOP16), U16 74HC595PW(TSSOP16), U17 74HC595PW(TSSOP16), U18 74HC595PW(TSSOP16), U19 74HC595PW(TSSOP16), U2 TPS2553DBVR(SOT23-6), U3 INA180A2IDBVR(SOT23-5), U4 MCP1700T-3302E/TT(SOT23), U5 EFM8BB21F16G-C(QSOP24), U6 PE42520C-Z(QFN16), U7 PE42520C-Z(QFN16), U8 PE42582A(QFN24), U9 NA(PE42520C-Z)

Commit message: PCB: routed board, 100 x 104 mm, DRC clean, JLC DFM only the exposed-pad vias
KiCad DRC: 0 errors, 0 unconnected, 0 schematic parity (warnings only: library
footprint mismatch, silk overlap/edge). JLC DFM: via-pad FAIL only on the 35
thermal vias in the QFN exposed pads (accepted), 26 WARN at 0.10-0.15 mm.
Project file: every netclass clearance 0.15 mm (the committed file was stale).

Co-Authored-By: Claude Opus 5.5 <noreply@anthropic.com>
Claude-Session: https://claude.ai/code/session_01YRUiF8Vp4242sya9Xyg3TV
Parts:
- L6: value 10uH/0805 -> 10uH/0.45A(1210); footprint Inductor_SMD:L_0805_2012Metric -> Inductor_SMD:L_1210_3225Metric
- moved R11 40.0 mm to (125.5, 127.2), turned to 90 degrees
- moved R3 16.8 mm to (141.2, 82.8), turned to 0 degrees
- moved D3 15.7 mm to (124.2, 142.0)
- moved R12 15.6 mm to (126.5, 89.0), turned to 180 degrees
- moved C27 15.0 mm to (78.8, 130.8)
- moved L3 14.8 mm to (78.0, 133.8)
- moved TP6 14.2 mm to (130.5, 84.8)
- moved R9 13.4 mm to (121.2, 140.5)
- moved C15 11.2 mm to (130.8, 95.5), turned to -90 degrees
- moved R19 9.00 mm to (144.0, 95.8)
- moved R20 5.49 mm to (61.0, 70.2)
- moved L6 4.78 mm to (141.5, 109.2), turned to 90 degrees
- moved R13 4.51 mm to (134.2, 98.0)
- moved C13 4.24 mm to (113.0, 141.0), turned to -90 degrees
- moved C6 3.18 mm to (110.0, 138.0)
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Routing:
- net Net-(D34-K): track 0.00 -> 1.74 mm, vias 0 -> 1
- net Net-(D10-K): track 0.00 -> 1.74 mm, vias 0 -> 1
- net Net-(D50-K): track 0.00 -> 1.74 mm, vias 0 -> 1
- net Net-(D49-K): track 0.00 -> 1.74 mm, vias 0 -> 1
- net Net-(D45-K): track 0.00 -> 1.74 mm, vias 0 -> 1
- net Net-(D44-K): track 0.00 -> 1.74 mm, vias 0 -> 1
- net Net-(D40-K): track 0.00 -> 1.74 mm, vias 0 -> 1
- net Net-(D39-K): track 0.00 -> 1.74 mm, vias 0 -> 1
- net Net-(D35-K): track 0.00 -> 1.74 mm, vias 0 -> 1
- net Net-(D26-K): track 0.00 -> 1.74 mm, vias 0 -> 1
- net Net-(D25-K): track 0.00 -> 1.74 mm, vias 0 -> 1
- net Net-(D21-K): track 0.00 -> 1.74 mm, vias 0 -> 1
- net Net-(D20-K): track 0.00 -> 1.74 mm, vias 0 -> 1
- net Net-(D16-K): track 0.00 -> 1.74 mm, vias 0 -> 1
- net Net-(D15-K): track 0.00 -> 1.74 mm, vias 0 -> 1
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Other:
- board size 100 x 102 mm -> 100 x 104 mm

Commit message: PCB rev with EFM8 QFN20, BWSMA-KE-P001 air launch, Brightking GDT: routed, DRC clean, JLC package
Routed on the G7 with srouter feat/cuda-wavefront; U5 fan-out ring; one duplicate SW_V1 via merged,
one strip via nudged 0.027 mm off U17.1. KiCad DRC: 0 errors, 0 unconnected, 0 schematic parity.
JLC DFM: via-pad FAIL only on the 38 exposed-pad thermal vias (accepted). Pours keep 0.3 mm from the
SMA notch walls on all layers (new .kicad_dru). JLC: 85 BOM lines, 217 placed, 9 not assembled;
jlc_rotfix 215 OK, J2/J3 set by cpl_override.py (EasyEDA origin 2.70 mm inside, body out).
Stock at JLC tonight: PE42582A-X 3 (one board), PE42520C-Z 8, RS-06MR390FT 13; everything else >= 60.

Co-Authored-By: Claude Opus 5.5 <noreply@anthropic.com>
Claude-Session: https://claude.ai/code/session_01YRUiF8Vp4242sya9Xyg3TV
Parts:
- removed TP1: TP/TX, TestPoint:TestPoint_Pad_D1.0mm
- added R30: 1k/1%, Resistor_SMD:R_0603_1608Metric, F.Cu at (143.2, 93.8)
- C701, C703: value 8.2pF/50V/C0G -> 12pF/50V/C0G
- C702: value 4.7pF/50V/C0G -> 6.8pF/50V/C0G
- GDT1: value 4532-090V(1812) -> 4532-091-LF(1812)
- J2, J3: footprint Connector_Coaxial:SMA_Amphenol_132289_EdgeMount -> coaxolotl:SMA_EdgeLaunch_BWSMA-KE-P001_Air
- L701, L702: value 15nH/5% -> 10nH/5%
- U5: value EFM8BB21F16G-C(QSOP24) -> EFM8BB21F16G-C(QFN20); footprint Package_SO:QSOP-24_3.9x8.7mm_P0.635mm -> coaxolotl:EFM8_QFN-20-1EP_3x3mm_P0.5mm_EP1.7x1.7mm
- moved R3 17.0 mm to (132.0, 97.0)
- moved TP6 16.3 mm to (142.0, 96.2)
- moved C27 15.0 mm to (63.8, 130.8)
- moved L3 14.8 mm to (64.5, 127.8)
- moved C2 14.6 mm to (135.0, 96.2), turned to -90 degrees
- moved R24 13.5 mm to (146.8, 117.8)
- moved L6 13.3 mm to (146.8, 121.5)
- moved R13 11.1 mm to (143.2, 91.5), turned to 0 degrees
- moved R16 9.18 mm to (136.0, 84.5), turned to 180 degrees
- moved C15 8.78 mm to (139.5, 96.2)
- moved R4 8.71 mm to (131.5, 85.8), turned to 90 degrees
- moved R17 7.98 mm to (139.8, 84.5)
- moved C14 7.91 mm to (137.2, 96.2)
- moved R12 7.07 mm to (131.5, 94.0), turned to -90 degrees
- moved R18 5.06 mm to (143.2, 88.5)
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Connections:
- J1 pad 2: Net-(J1-Pin_2) -> /MCU/C2D
- U5 pad 1: Net-(U5-P0.3/ADC) -> /MCU/SENSE
- U5 pad 10: /MCU/LED_RCK -> /MCU/LNA_PATH_OUT
- U5 pad 11: /MCU/LED_SCK -> /Filter bank/SW_V3
- U5 pad 12: /MCU/LED_SER -> GND
- U5 pad 13: unconnected-(U5-P1.7-Pad13) -> /Filter bank/SW_V2
- U5 pad 14: unconnected-(U5-P1.6-Pad14) -> /Filter bank/SW_V1
- U5 pad 15: unconnected-(U5-P1.5-Pad15) -> /MCU/LNA_PATH
- U5 pad 16: /MCU/LNA_PATH_OUT -> /MCU/LNA_EN
- U5 pad 17: /MCU/FMN -> /MCU/FAULT_N
- U5 pad 18: /Filter bank/SW_V3 -> /MCU/LED_OE_N
- U5 pad 19: /Filter bank/SW_V2 -> Net-(U5-P0.3/ADC)
- U5 pad 2: /MCU/SCAP_ADC -> /MCU/SENSE
- U5 pad 20: /Filter bank/SW_V1 -> /MCU/SCAP_ADC
- U5 pad 21: /MCU/LNA_PATH -> GND
- U5 pad 3: /MCU/SENSE -> GND
- U5 pad 4: /MCU/SENSE -> +3V3
- U5 pad 5: GND -> Net-(J1-Pin_3)
- U5 pad 6: +3V3 -> /MCU/C2D
- U5 pad 7: Net-(J1-Pin_3) -> /MCU/LED_RCK
- U5 pad 8: Net-(J1-Pin_2) -> /MCU/LED_SCK
- U5 pad 9: /MCU/LED_OE_N -> /MCU/LED_SER
Routing:
- net /MCU/SENSE: track 0.00 -> 2.80 mm, vias 0 -> 2
- net /MCU/SCAP_ADC: track 0.00 -> 1.80 mm, vias 0 -> 1
- net /MCU/LNA_PATH_OUT: track 1.00 -> 2.80 mm, vias 1 -> 2
- net /MCU/LED_SCK: track 8.00 -> 9.80 mm, vias 0 -> 1
- net /MCU/LED_OE_N: track 8.00 -> 9.80 mm, vias 0 -> 1
- net /MCU/C2D: track 0.00 -> 1.80 mm, vias 0 -> 1
- net /MCU/LNA_PATH: track 1.00 -> 2.80 mm, vias 1 -> 2
- net /Filter bank/SW_V2: track 2.00 -> 3.80 mm, vias 2 -> 3
- net Net-(U5-P0.3/ADC): track 0.00 -> 1.00 mm, vias 0 -> 1
- net Net-(J1-Pin_3): track 0.00 -> 1.00 mm, vias 0 -> 1
- net /MCU/LNA_EN: track 0.00 -> 1.00 mm, vias 0 -> 1
- net /MCU/LED_SER: track 8.00 -> 9.00 mm, vias 0 -> 1
- net /MCU/LED_RCK: track 8.00 -> 9.00 mm, vias 0 -> 1
- net /MCU/FAULT_N: track 0.00 -> 1.00 mm, vias 0 -> 1
- net /Filter bank/SW_V3: track 3.60 -> 4.60 mm, vias 2 -> 3
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Other:
- outline, holes or cut-outs redrawn
